File: board/openzone.kicad_pcb (KiCad board)
At the start: 2 copper layers, 97.8 x 76.2 mm, 28 parts, among them J1 Motor1, J10 AC serial, J11 Power Supply, J12 Step Down Power Supply, J13 Motor Power Supply Selector, J2 Motor2, J3 Motor3, J4 Motor4, J5 Motor5, J6 Motor6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

Commit message: A lot of changes
Including:

* ESP32 relocation to improve WiFi signal strength.
* Voltage divider for serial TTL communication with Air Conditioner.
* New PCB terminals footprint. My own.
* Adds OpenZone logo.
Parts:
- added R2: 4,7K, Resistor_THT:R_Axial_DIN0207_L6.3mm_D2.5mm_P7.62mm_Horizontal, F.Cu at (180.8, 130.5)
- added R3: 10K, Resistor_THT:R_Axial_DIN0207_L6.3mm_D2.5mm_P7.62mm_Horizontal, F.Cu at (183.9, 130.5)
- J1, J2, J3, J4, J5, J6, J7, J8: footprint TerminalBlock_Phoenix:TerminalBlock_Phoenix_MKDS-1,5-2_1x02_P5.00mm_Horizontal -> SKaRCHa:KF301-2P-5
- J9: footprint SKaRCHa:WEMOS_D1_MINI32 -> SKaRCHa:WEMOS_D1_MINI32_UP
- moved REF** 45.7 mm to (156.8, 106.0), turned to 0 degrees
- moved REF** 34.3 mm to (156.8, 114.3)
- moved J9 26.3 mm to (174.7, 132.9), turned to 180 degrees
- moved J8 7.30 mm to (191.8, 68.3), turned to 0 degrees
- moved J7 6.74 mm to (180.3, 68.3), turned to 0 degrees
- moved J6 6.17 mm to (168.9, 68.3), turned to 0 degrees
- moved J11 6.10 mm to (115.6, 122.9)
- moved J13 6.10 mm to (113.0, 115.3)
- moved J12 6.10 mm to (129.5, 128.0)
- moved J5 5.61 mm to (157.5, 68.3), turned to 0 degrees
- moved J4 5.05 mm to (146.1, 68.3), turned to 0 degrees
- moved J3 4.50 mm to (134.6, 68.3), turned to 0 degrees
- moved J2 3.94 mm to (123.2, 68.3), turned to 0 degrees
- moved J10 3.70 mm to (139.1, 107.3)
- moved J1 3.40 mm to (111.8, 68.3), turned to 0 degrees
Connections:
- J10 pad 2: IO16_RX -> Net-(J10-Pad2)
- U1 pad 10: IO12 -> IO32
- U1 pad 11: Net-(J2-Pad1) -> Net-(J2-Pad2)
- U1 pad 14: Net-(J2-Pad2) -> Net-(J2-Pad1)
- U1 pad 15: IO32 -> IO12
- U1 pad 2: IO04 -> IO25
- U1 pad 3: Net-(J1-Pad1) -> Net-(J1-Pad2)
- U1 pad 6: Net-(J1-Pad2) -> Net-(J1-Pad1)
- U1 pad 7: IO02 -> IO27
- U2 pad 10: IO22 -> IO15
- U2 pad 11: Net-(J4-Pad1) -> Net-(J4-Pad2)
- U2 pad 14: Net-(J4-Pad2) -> Net-(J4-Pad1)
- U2 pad 2: IO27 -> IO02
- U2 pad 3: Net-(J3-Pad1) -> Net-(J3-Pad2)
- U2 pad 6: Net-(J3-Pad2) -> Net-(J3-Pad1)
- U2 pad 7: IO25 -> IO04
- U3 pad 10: IO05 -> IO18
- U3 pad 11: Net-(J6-Pad1) -> Net-(J6-Pad2)
- U3 pad 14: Net-(J6-Pad2) -> Net-(J6-Pad1)
- U3 pad 15: IO23 -> IO19
- U3 pad 2: IO14 -> IO26
- U3 pad 3: Net-(J5-Pad1) -> Net-(J5-Pad2)
- U3 pad 6: Net-(J5-Pad2) -> Net-(J5-Pad1)
- U3 pad 7: IO15 -> IO22
- U4 pad 10: IO33 -> IO14
- U4 pad 11: Net-(J8-Pad1) -> Net-(J8-Pad2)
- U4 pad 14: Net-(J8-Pad2) -> Net-(J8-Pad1)
- U4 pad 15: IO26 -> IO33
- U4 pad 2: IO19 -> IO05
- U4 pad 3: Net-(J7-Pad1) -> Net-(J7-Pad2)
- U4 pad 6: Net-(J7-Pad2) -> Net-(J7-Pad1)
- U4 pad 7: IO18 -> IO23
Routing:
- net Net-(J10-Pad2): track 0.00 -> 57.0 mm
- net IO14: track 73.0 -> 25.6 mm
- net IO25: track 35.3 -> 78.5 mm
- net IO16_RX: track 44.8 -> 14.0 mm
- net IO04: track 70.4 -> 43.4 mm
- net IO27: track 45.0 -> 68.7 mm
- net +5V: track 245.8 -> 222.2 mm
- net IO21: track 45.2 -> 66.4 mm
- net IO26: track 36.1 -> 56.2 mm
- net IO17_TX: track 37.7 -> 56.3 mm
- net IO23: track 45.8 -> 27.1 mm
- net IO33: track 26.4 -> 43.9 mm
- net IO12: track 50.9 -> 65.3 mm
- net IO18: track 26.0 -> 37.8 mm
- net Net-(J4-Pad1): track 29.0 -> 18.3 mm
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Other:
- board size 97.8 x 76.2 mm -> 97.8 x 78.5 mm
- board text added: "OpenZone"
- board text added: "Version 1.0"
